File: hw/qfmu/sensors.kicad_sch (KiCad schematic)
At the start: 7 parts, among them U15 BMI088

Commit message: feat: add new BLDC controler and RF section
Other:
- company: Daniel Pérez -> Daniel Enrique Pérez Díaz
- title: (none) -> Quincy FMU
Changed lines of the file:
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@@
 	(paper "A4")
 	(title_block
-		(date "2024-09-10")
+		(title "Quincy FMU")
+		(date "2024-09-28")
 		(rev "0")
-		(company "Daniel Pérez")
+		(company "Daniel Enrique Pérez Díaz")
+		(comment 1 "Flight Management Unit for the Quincy Quadcopter project.")
 	)
 	(junction
