File: hw/qfmu/qfmu.kicad_pcb (KiCad board)
At the start: 2 copper layers, 208 parts, among them J1 Conn_02x06_Counter_Clockwise, J2 Conn_Coaxial, J3 Conn_01x03_Pin, J4 Conn_01x03_Pin, J5 Conn_01x03_Pin, J6 Conn_01x03_Pin, Q1 IRF540N, Q10 IRF540N, Q11 IRF540N, Q12 IRF540N, Q13 IRF540N, Q14 IRF540N, Q15 IRF540N, Q16 IRF540N, Q17 IRF540N, Q18 IRF540N, Q19 IRF540N, Q2 IRF540N, Q20 IRF540N, Q21 IRF540N, Q22 IRF540N, Q23 IRF540N, Q24 IRF540N, Q25 AO3401A, Q26 AO3400A, Q27 IRF540N, Q29 IRF540N, Q3 IRF540N, Q30 IRF540N, Q31 IRF540N, Q4 IRF540N, Q5 IRF540N, Q6 IRF540N, Q7 IRF540N, Q8 IRF540N, Q9 IRF540N, U1 EFM32GG11B120F2048GQ64, U12 AS179-92LF, U14 TPS562202, Y1 Crystal_GND24, Y2 Crystal, Y3 13.52 MHz, Y4 13.52 MHz

Commit message: feat: start PCB design, define board outline and basic placement
Parts:
- added FUSE1: ITV5432L5030WR, ITV5432:QFN4_ITV5432_LTF, F.Cu at (160.6, 89.7)
- added J7: Conn_02x06_Counter_Clockwise, Connector_PinHeader_2.54mm:PinHeader_2x06_P2.54mm_Vertical, F.Cu at (96.9, 109.7)
- added Q28: FCX495TA, FCX495TA:SOT89_DIO, F.Cu at (219.3, 113.9)
- added REF**: BatteryHolder_Keystone_1042_1x18650, Battery:BatteryHolder_Keystone_1042_1x18650, F.Cu at (155.4, 148.1)
- added REF**: BatteryHolder_Keystone_1042_1x18650, Battery:BatteryHolder_Keystone_1042_1x18650, F.Cu at (155.4, 169.7)
- added REF**: BatteryHolder_Keystone_1042_1x18650, Battery:BatteryHolder_Keystone_1042_1x18650, F.Cu at (155.4, 126.5)
- added TP10: TestPoint, Connector_Pin:Pin_D0.7mm_L6.5mm_W1.8mm_FlatFork, F.Cu at (191.2, 92.0)
- added TP11: TestPoint, Connector_Pin:Pin_D0.7mm_L6.5mm_W1.8mm_FlatFork, F.Cu at (112.1, 191.2)
- added TP12: TestPoint, Connector_Pin:Pin_D0.7mm_L6.5mm_W1.8mm_FlatFork, F.Cu at (218.3, 180.1)
- added TP5: TestPoint, Connector_Pin:Pin_D0.7mm_L6.5mm_W1.8mm_FlatFork, F.Cu at (128.0, 92.5)
- added TP6: TestPoint, Connector_Pin:Pin_D0.7mm_L6.5mm_W1.8mm_FlatFork, F.Cu at (191.2, 88.6)
- added TP7: TestPoint, Connector_Pin:Pin_D0.7mm_L6.5mm_W1.8mm_FlatFork, F.Cu at (112.1, 187.7)
- added TP8: TestPoint, Connector_Pin:Pin_D0.7mm_L6.5mm_W1.8mm_FlatFork, F.Cu at (218.3, 176.6)
- added TP9: TestPoint, Connector_Pin:Pin_D0.7mm_L6.5mm_W1.8mm_FlatFork, F.Cu at (128.0, 96.0)
- added U10: BQ7694202PFBR, BQ76942:PFB0048A_N, F.Cu at (208.7, 114.5)
- added U11: MICRF219AAYQS-TR, MICRF219:QSOP16_MC_MCH, F.Cu at (179.0, 208.0)
- added U13: MICRF113YM6-TR, MICRF113:SOT-23-6_MC_MCH, F.Cu at (155.8, 202.2)
- added U15: BMI088, BMI088:PQFN50P450X300X100-16N, F.Cu at (159.8, 195.1)
- added U2: DRV8300UDPWR, DRV8300:TSSOP_0DIPWR_TEX, F.Cu at (106.0, 82.3)
- added U3: DRV8300UDPWR, DRV8300:TSSOP_0DIPWR_TEX, F.Cu at (205.5, 83.3)
- added U4: DRV8300UDPWR, DRV8300:TSSOP_0DIPWR_TEX, F.Cu at (105.4, 210.8)
- added U5: DRV8300UDPWR, DRV8300:TSSOP_0DIPWR_TEX, F.Cu at (208.7, 208.3)
- added U6: IMC101TT038XUMA1, IMC101TT038XUMA1:SOP50P640X110-38N, F.Cu at (91.8, 98.0)
- added U7: IMC101TT038XUMA1, IMC101TT038XUMA1:SOP50P640X110-38N, F.Cu at (220.9, 97.5)
- added U8: IMC101TT038XUMA1, IMC101TT038XUMA1:SOP50P640X110-38N, F.Cu at (92.2, 196.7)
- added U9: IMC101TT038XUMA1, IMC101TT038XUMA1:SOP50P640X110-38N, F.Cu at (222.4, 195.7)
- U1: footprint EFM32GG11B120F2048GQ64:TQFP64_10X10_SIL -> EFM32GG11B120F:TQFP64_10X10_SIL
- moved J6 256.4 mm to (255.3, 249.1), turned to 45 degrees
- moved Q4 239.1 mm to (233.5, 235.1), turned to -135 degrees
- moved J4 230.8 mm to (259.4, 49.8), turned to 135 degrees
- moved Q8 230.6 mm to (242.5, 226.4), turned to -135 degrees
- moved Q12 221.8 mm to (251.4, 217.5), turned to -135 degrees
- moved Q16 216.5 mm to (225.3, 234.1), turned to 45 degrees
- moved Q20 207.4 mm to (234.2, 225.2), turned to 45 degrees
- moved Q2 203.6 mm to (228.0, 54.4), turned to -45 degrees
- moved Q6 202.3 mm to (237.4, 62.6), turned to -45 degrees
- moved Q10 200.9 mm to (246.3, 71.5), turned to -45 degrees
- moved Q24 198.2 mm to (243.1, 216.3), turned to 45 degrees
- moved Y3 186.5 mm to (187.8, 203.1), turned to 90 degrees
- moved D4 184.2 mm to (218.8, 206.8), turned to 45 degrees
- moved D2 177.1 mm to (217.8, 85.9), turned to -45 degrees
- moved R12 174.1 mm to (187.5, 108.6)
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Connections:
- TP1 pad 1: /Motor 1/MOTOR_SPEED -> /Microcontroller/MOTOR_SPEED1
- TP2 pad 1: /Motor 2/MOTOR_SPEED -> /Microcontroller/MOTOR_SPEED2
- TP3 pad 1: /Motor 3/MOTOR_SPEED -> /Microcontroller/MOTOR_SPEED3
- TP4 pad 1: /Motor 4/MOTOR_SPEED -> /Microcontroller/MOTOR_SPEED4
- U1 pad 1: unconnected-(U1-PA0-Pad1) -> /Microcontroller/MOTOR_SPEED1
- U1 pad 10: unconnected-(U1-PC1-Pad10) -> /Microcontroller/DIR2
- U1 pad 11: unconnected-(U1-PC2-Pad11) -> /Microcontroller/DIR3
- U1 pad 12: unconnected-(U1-PC3-Pad12) -> /Microcontroller/DIR4
- U1 pad 2: unconnected-(U1-PA1-Pad2) -> /Microcontroller/MOTOR_SPEED2
- U1 pad 28: unconnected-(U1-PD0-Pad28) -> /Microcontroller/DUTY1
- U1 pad 29: unconnected-(U1-PD1-Pad29) -> /Microcontroller/DUTY2
- U1 pad 3: unconnected-(U1-PA2-Pad3) -> /Microcontroller/MOTOR_SPEED3
- U1 pad 30: unconnected-(U1-PD2-Pad30) -> /Microcontroller/DUTY3
- U1 pad 31: unconnected-(U1-PD3-Pad31) -> /Microcontroller/DUTY4
- U1 pad 36: unconnected-(U1-PD8-Pad36) -> /Microcontroller/RF_DEMOD
- U1 pad 37: unconnected-(U1-PC6-Pad37) -> /Microcontroller/TX_ASK
- U1 pad 38: unconnected-(U1-PC7-Pad38) -> /Microcontroller/ANT_MODE
- U1 pad 4: unconnected-(U1-PA3-Pad4) -> /Microcontroller/MOTOR_SPEED4
- U1 pad 5: unconnected-(U1-PA4-Pad5) -> /Microcontroller/IMU_INT_AC1
- U1 pad 59: unconnected-(U1-PE10-Pad59) -> /Microcontroller/MON_ALERT
- U1 pad 6: unconnected-(U1-PA5-Pad6) -> /Microcontroller/IMU_INT_GY1
- U1 pad 60: unconnected-(U1-PE11-Pad60) -> /Power/MON_SDA
- U1 pad 61: unconnected-(U1-PE12-Pad61) -> /Power/MON_SCL
- U1 pad 62: unconnected-(U1-PE13-Pad62) -> /Microcontroller/DCHG
- U1 pad 63: unconnected-(U1-PE14-Pad63) -> /Microcontroller/DDSG
- U1 pad 64: unconnected-(U1-PE15-Pad64) -> /Microcontroller/MON_RST_SHUT
- U1 pad 9: unconnected-(U1-PC0-Pad9) -> /Microcontroller/DIR1
Routing:
- net /Motor 2/LO3: track 0.00 -> 37.8 mm, vias 0 -> 1
- net /Motor 1/LO3: track 0.00 -> 5.94 mm
- net /Motor 1/OUTA: track 0.00 -> 5.94 mm
- net /Motor 1/LO2: track 0.00 -> 5.37 mm
Other:
- board outline added: 246 x 244 mm
- copper layers 2 -> 4

Commit message: feat: complete preliminar placement of PCB components
Organize and place components for routing and export a preliminary BOM
Parts:
- added L5: IND_VLS5045EX-3R3N, VLS5045EX_3R3N:IND_VLS5045EX-3R3N, F.Cu at (129.5, 94.0)
- C20, C37, C38, C39, C41, C48, C49, C5, C50, C56, C6, C60, C74, C75, C82, C84, C91, Q25, Q26, R2, R24, R29, R30, R31, R34, R4, R41, R42, R44, R45, R48, R49, R53, R57: moved to B.Cu
- moved J1 112.3 mm to (161.3, 106.4), turned to -90 degrees
- moved U12 111.9 mm to (159.5, 198.4), turned to -90 degrees
- moved L1 104.3 mm to (148.9, 203.0)
- moved Q25 97.3 mm to (158.3, 198.9), turned to 180 degrees
- moved Q26 96.0 mm to (158.3, 202.4), turned to 180 degrees
- moved L3 95.3 mm to (149.1, 195.9), turned to -90 degrees
- moved R33 82.9 mm to (220.0, 144.0), turned to -90 degrees
- moved R34 81.5 mm to (214.9, 152.9), turned to -90 degrees
- moved R32 79.9 mm to (214.9, 144.0), turned to 90 degrees
- moved TH2 75.1 mm to (163.4, 181.4)
- moved R24 74.5 mm to (210.1, 124.0), turned to 90 degrees
- moved R25 71.3 mm to (206.0, 129.8)
- moved R21 71.0 mm to (201.3, 129.8)
- moved R39 70.3 mm to (221.0, 118.4), turned to -90 degrees
- moved R28 68.9 mm to (210.8, 107.2), turned to 90 degrees
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- renumbered REF** to CELL1, REF** to CELL2, REF** to CELL3
Connections:
- CELL1 pad 1: (no net) -> /Power/VCELL3
- CELL1 pad 2: (no net) -> /Power/VCELL2
- CELL2 pad : (no net) -> /Power/VCELL2
- CELL2 pad 2: (no net) -> /Power/VCELL1
- CELL3 pad 1: (no net) -> /Power/VCELL1
- CELL3 pad 2: (no net) -> /Power/PACK_NEG
Routing:
- net /Motor 2/LO3: track 37.8 -> 0.00 mm, vias 1 -> 0
- net /Motor 1/LO3: track 5.94 -> 0.00 mm
- net /Motor 1/OUTA: track 5.94 -> 0.00 mm
- net /Power/VCELL2: track 0.00 -> 5.90 mm
- net /Power/VCELL1: track 0.00 -> 5.88 mm
- net /Power/PACK_NEG: track 0.00 -> 5.73 mm
- net /Power/VCELL3: track 0.00 -> 5.66 mm
- net /Motor 1/LO2: track 5.37 -> 0.00 mm
- net Net-(D1-A): track 0.00 -> 3.57 mm
- net +12V: track 0.00 -> 2.70 mm, vias 0 -> 1
- net /Motor 1/PWM_WH: track 0.00 -> 0.93 mm
- added copper zone on In2.Cu, net GND
Other:
- board text added: "+3.3V"
- board text added: "BLDC FW UART"
- board text added: "DNP"
- board text added: "Daniel Enrique Pérez Díaz"
- board text added: "GND"
- board text added: "JTAG/SWD"
- board text added: "RSTN"
- board text added: "RX1"
- board text added: "RX2"
- board text added: "RX3"
- board text added: "RX4"
- board text added: "SWCK/ TCLK"
- board text added: "SWO/ TDO"
- board text added: "TDI"
- board text added: "TMS/ SWDIO"
- board text added: "TX1"
- board text added: "TX2"
- board text added: "TX3"
- board text added: "TX4"

Commit message: feat: add basic split power planes and redo edgecuts
Add power plane zones and fix edgecuts constraints, also reducing the size.
Parts:
- moved C71 56.2 mm to (180.8, 97.2)
- moved C67 56.2 mm to (187.6, 107.9)
- moved C70 56.2 mm to (191.6, 110.3)
- moved C72 56.2 mm to (189.5, 97.5)
- moved L5 56.2 mm to (185.2, 102.1)
- moved R36 56.2 mm to (194.7, 107.2)
- moved R37 56.2 mm to (194.7, 105.1)
- moved R38 56.2 mm to (190.6, 103.7)
- moved C68 56.2 mm to (183.2, 107.9)
- moved C69 56.2 mm to (185.4, 107.9)
- moved U14 56.2 mm to (190.7, 107.2)
- moved J7 24.4 mm to (166.4, 111.8), turned to 180 degrees
- moved J1 24.3 mm to (138.2, 99.1), turned to 0 degrees
- moved R43 14.3 mm to (101.4, 105.9)
- moved C73 14.3 mm to (103.6, 105.9)
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Routing:
- net Net-(D1-A): track 3.57 -> 0.00 mm
- added copper zone on In1.Cu, net +12V
- added copper zone on In1.Cu, net +3.3V
- removed copper zone on In2.Cu, net GND
Other:
- board size 246 x 244 mm -> 244 x 244 mm
- board text added: "MOTOR 1"
- board text added: "MOTOR 2"
- board text added: "MOTOR 3"
- board text added: "MOTOR 4"

Commit message: feat: further routing
Parts:
- moved R6 86.7 mm to (177.0, 192.8), turned to -90 degrees
- moved R5 80.2 mm to (174.8, 189.8), turned to -90 degrees
- moved FUSE1 38.1 mm to (202.9, 101.2)
- moved D5 24.9 mm to (196.7, 111.5), turned to 180 degrees
- moved R25 18.9 mm to (201.2, 111.5)
- moved Y1 10.6 mm to (113.9, 205.1)
- moved R51 4.11 mm to (108.4, 91.7), turned to 180 degrees
- moved C64 3.94 mm to (214.9, 128.8)
- moved C4 3.62 mm to (120.9, 204.2)
- moved C3 3.62 mm to (120.9, 206.2)
- moved C5 3.34 mm to (117.6, 202.2), turned to -90 degrees
- moved C29 2.64 mm to (102.9, 96.8)
- moved C67 2.60 mm to (185.7, 109.7)
- moved C68 2.60 mm to (181.4, 109.7)
- moved C69 2.60 mm to (183.5, 109.7)
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Connections:
- L5 pad 1: (no net) -> +3.3V
- L5 pad 2: (no net) -> Net-(U14-SW)
Routing:
- net /Power/CMN_DRAIN: track 0.00 -> 174.7 mm, vias 0 -> 7
- net /Power/MON_SDA: track 0.00 -> 164.3 mm, vias 0 -> 2
- net /Microcontroller/MON_RST_SHUT: track 0.00 -> 164.0 mm, vias 0 -> 4
- net /Microcontroller/DDSG: track 0.00 -> 161.4 mm, vias 0 -> 2
- net /Power/VCELL3: track 5.66 -> 165.9 mm, vias 0 -> 2
- net /Microcontroller/DCHG: track 0.00 -> 158.6 mm, vias 0 -> 2
- net /Power/MON_SCL: track 0.00 -> 146.9 mm
- net /Microcontroller/MON_ALERT: track 0.00 -> 145.5 mm, vias 0 -> 2
- net GND: track 0.00 -> 132.1 mm, vias 0 -> 65
- net Net-(Q27-G): track 0.00 -> 125.9 mm, vias 0 -> 2
- net /Microcontroller/RESETN: track 0.00 -> 125.0 mm, vias 0 -> 4
- net Net-(Q29-G): track 0.00 -> 122.7 mm, vias 0 -> 1
- net /Microcontroller/DUTY1: track 0.00 -> 119.8 mm, vias 0 -> 2
- net /Microcontroller/MOTOR_SPEED1: track 0.00 -> 116.9 mm, vias 0 -> 1
- net /Microcontroller/DIR1: track 0.00 -> 114.6 mm, vias 0 -> 2
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- added copper zone on In2.Cu, net GND

Commit message: feat: reposition elements and go back to original edgecuts
Position elements for easier routing and start from scratch.
Revert shape design to be fully symmetrical.
Parts:
- added PWRIN1: TestPoint, Connector_Pin:Pin_D0.7mm_L6.5mm_W1.8mm_FlatFork, F.Cu at (192.5, 95.8)
- C20, C37, C38, C39, C41, C48, C49, C5, C50, C56, C6, C60, C74, C75, C82, C84, C91, Q25, Q26, R2, R24, R29, R30, R31, R34, R4, R41, R42, R44, R45, R48, R49, R53, R57: moved to F.Cu
- moved C62 111.8 mm to (96.5, 116.9), turned to 90 degrees
- moved C66 111.3 mm to (109.2, 116.9)
- moved U10 110.6 mm to (98.8, 127.8)
- moved R40 110.6 mm to (110.1, 131.0)
- moved R39 110.6 mm to (108.1, 131.0)
- moved R24 110.3 mm to (100.8, 139.6)
- moved R27 110.1 mm to (92.7, 139.6), turned to 90 degrees
- moved C65 110.0 mm to (105.2, 133.1), turned to 90 degrees
- moved C61 109.7 mm to (94.5, 116.9), turned to -90 degrees
- moved Q28 109.7 mm to (108.2, 126.0), turned to -90 degrees
- moved R29 109.7 mm to (100.6, 116.9)
- moved R28 108.6 mm to (102.6, 116.9)
- moved C59 108.1 mm to (98.8, 139.7)
- moved C60 108.0 mm to (98.6, 116.9), turned to -90 degrees
- moved R26 107.5 mm to (94.7, 139.6), turned to 90 degrees
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Routing:
- net /Power/CMN_DRAIN: track 174.7 -> 0.00 mm, vias 7 -> 0
- net /Power/VCELL3: track 165.9 -> 0.00 mm, vias 2 -> 0
- net /Power/MON_SDA: track 164.3 -> 0.00 mm, vias 2 -> 0
- net /Microcontroller/MON_RST_SHUT: track 164.0 -> 0.00 mm, vias 4 -> 0
- net /Microcontroller/DDSG: track 161.4 -> 0.00 mm, vias 2 -> 0
- net /Microcontroller/DCHG: track 158.6 -> 0.00 mm, vias 2 -> 0
- net /Power/MON_SCL: track 146.9 -> 0.00 mm
- net /Microcontroller/MON_ALERT: track 145.5 -> 0.00 mm, vias 2 -> 0
- net GND: track 132.1 -> 0.00 mm, vias 65 -> 0
- net Net-(Q27-G): track 125.9 -> 0.00 mm, vias 2 -> 0
- net /Microcontroller/RESETN: track 125.0 -> 0.00 mm, vias 4 -> 0
- net Net-(Q29-G): track 122.7 -> 0.00 mm, vias 1 -> 0
- net /Microcontroller/DUTY1: track 119.8 -> 0.00 mm, vias 2 -> 0
- net /Microcontroller/MOTOR_SPEED1: track 116.9 -> 0.00 mm, vias 1 -> 0
- net /Microcontroller/DIR1: track 114.6 -> 0.00 mm, vias 2 -> 0
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Other:
- outline, holes or cut-outs redrawn
